File: pcb/Uhrbox-E-plugboard.sch (KiCad schematic (older format))
At the start: 21 parts, among them J1 Conn_01x20_Female, J10 Conn_01x01_MountingPin, J11 Conn_01x01_MountingPin, J13 Conn_01x01_MountingPin, J14 Conn_01x01_MountingPin, J15 Conn_01x01_MountingPin, J16 Conn_01x01_MountingPin, J17 Conn_01x01_MountingPin, J18 Conn_01x01_MountingPin, J19 Conn_01x01_MountingPin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

Commit message: Uhrbord-E plugboard PCB sent to manufacturing
Parts:
- added H1, H2, H3, H4, H5, H6: MountingHole_Pad, MountingHole:MountingHole_3.2mm_M3_Pad, symbol Mechanical:MountingHole_Pad
Connections:
- new net GND: H1.1, H2.1, H3.1, H4.1, H5.1, H6.1
Changed lines of the file:
@@
 Wire Wire Line
 	2050 3900 1500 3900
+$Comp
+L Mechanical:MountingHole_Pad H4
+U 1 1 5F692297
+P 10000 1050
+F 0 "H4" H 10100 1099 50  0000 L CNN
+F 1 "MountingHole_Pad" H 10100 1008 50  0000 L CNN
+F 2 "MountingHole:MountingHole_3.2mm_M3_Pad" H 10000 1050 50  0001 C CNN
+F 3 "~" H 10000 1050 50  0001 C CNN
+	1    10000 1050
+	1    0    0    -1
+$EndComp
+$Comp
+L Mechanical:MountingHole_Pad H5
+U 1 1 5F692F9B
+P 10000 1550
+F 0 "H5" H 10100 1599 50  0000 L CNN
+F 1 "MountingHole_Pad" H 10100 1508 50  0000 L CNN
+F 2 "MountingHole:MountingHole_3.2mm_M3_Pad" H 10000 1550 50  0001 C CNN
+F 3 "~" H 10000 1550 50  0001 C CNN
+	1    10000 1550
+	1    0    0    -1
+$EndComp
+$Comp
+L Mechanical:MountingHole_Pad H6
+U 1 1 5F6931A0
+P 10000 2050
+F 0 "H6" H 10100 2099 50  0000 L CNN
+F 1 "MountingHole_Pad" H 10100 2008 50  0000 L CNN
+F 2 "MountingHole:MountingHole_3.2mm_M3_Pad" H 10000 2050 50  0001 C CNN
+F 3 "~" H 10000 2050 50  0001 C CNN
+	1    10000 2050
+	1    0    0    -1
+$EndComp
+$Comp
+L Mechanical:MountingHole_Pad H1
+U 1 1 5F693397
+P 9000 1050
+F 0 "H1" H 9100 1099 50  0000 L CNN
+F 1 "MountingHole_Pad" H 9100 1008 50  0000 L CNN
+F 2 "MountingHole:MountingHole_3.2mm_M3_Pad" H 9000 1050 50  0001 C CNN
+F 3 "~" H 9000 1050 50  0001 C CNN
+	1    9000 1050
+	1    0    0    -1
+$EndComp
+$Comp
+L Mechanical:MountingHole_Pad H2
+U 1 1 5F693AA7
+P 9000 1550
+F 0 "H2" H 9100 1599 50  0000 L CNN
+F 1 "MountingHole_Pad" H 9100 1508 50  0000 L CNN
+F 2 "MountingHole:MountingHole_3.2mm_M3_Pad" H 9000 1550 50  0001 C CNN
+F 3 "~" H 9000 1550 50  0001 C CNN
+	1    9000 1550
+	1    0    0    -1
+$EndComp
+$Comp
+L Mechanical:MountingHole_Pad H3
+U 1 1 5F693E53
+P 9000 2050
+F 0 "H3" H 9100 2099 50  0000 L CNN
+F 1 "MountingHole_Pad" H 9100 2008 50  0000 L CNN
+F 2 "MountingHole:MountingHole_3.2mm_M3_Pad" H 9000 2050 50  0001 C CNN
+F 3 "~" H 9000 2050 50  0001 C CNN
+	1    9000 2050
+	1    0    0    -1
+$EndComp
+$Comp
+L power:GND #PWR01
+U 1 1 5F694481
+P 9000 1150
+F 0 "#PWR01" H 9000 900 50  0001 C CNN
+F 1 "GND" H 9005 977 50  0000 C CNN
+F 2 "" H 9000 1150 50  0001 C CNN
+F 3 "" H 9000 1150 50  0001 C CNN
+	1    9000 1150
+	1    0    0    -1
+$EndComp
+$Comp
+L power:GND #PWR04
+U 1 1 5F6947B2
+P 10000 1150
+F 0 "#PWR04" H 10000 900 50  0001 C CNN
+F 1 "GND" H 10005 977 50  0000 C CNN
+F 2 "" H 10000 1150 50  0001 C CNN
+F 3 "" H 10000 1150 50  0001 C CNN
+	1    10000 1150
+	1    0    0    -1
+$EndComp
+$Comp
+L power:GND #PWR05
+U 1 1 5F694BB3
+P 10000 1650
+F 0 "#PWR05" H 10000 1400 50  0001 C CNN
+F 1 "GND" H 10005 1477 50  0000 C CNN
+F 2 "" H 10000 1650 50  0001 C CNN
+F 3 "" H 10000 1650 50  0001 C CNN
+	1    10000 1650
+	1    0    0    -1
+$EndComp
+$Comp
+L power:GND #PWR06
+U 1 1 5F6950F8
+P 10000 2150
+F 0 "#PWR06" H 10000 1900 50  0001 C CNN
+F 1 "GND" H 10005 1977 50  0000 C CNN
+F 2 "" H 10000 2150 50  0001 C CNN
+F 3 "" H 10000 2150 50  0001 C CNN
+	1    10000 2150
+	1    0    0    -1
+$EndComp
+$Comp
+L power:GND #PWR03
+U 1 1 5F6953F5
+P 9000 2150
+F 0 "#PWR03" H 9000 1900 50  0001 C CNN
+F 1 "GND" H 9005 1977 50  0000 C CNN
+F 2 "" H 9000 2150 50  0001 C CNN
+F 3 "" H 9000 2150 50  0001 C CNN
+	1    9000 2150
+	1    0    0    -1
+$EndComp
+$Comp
+L power:GND #PWR02
+U 1 1 5F6956D3
+P 9000 1650
+F 0 "#PWR02" H 9000 1400 50  0001 C CNN
+F 1 "GND" H 9005 1477 50  0000 C CNN
+F 2 "" H 9000 1650 50  0001 C CNN
+F 3 "" H 9000 1650 50  0001 C CNN
+	1    9000 1650
+	1    0    0    -1
+$EndComp
 $EndSCHEMATC

Commit message: Changed header to 2.54mm and sent to manufacturing
Parts:
- J1: footprint Connector_PinHeader_2.00mm:PinHeader_1x20_P2.00mm_Vertical -> Connector_PinHeader_2.54mm:PinHeader_1x20_P2.54mm_Vertical
Changed lines of the file:
@@
 F 0 "J1" H 1192 3985 50  0000 C CNN
 F 1 "Conn_01x20_Female" H 1192 3894 50  0000 C CNN
-F 2 "Connector_PinHeader_2.00mm:PinHeader_1x20_P2.00mm_Vertical" H 1300 2900 50  0001 C CNN
+F 2 "Connector_PinHeader_2.54mm:PinHeader_1x20_P2.54mm_Vertical" H 1300 2900 50  0001 C CNN
 F 3 "~" H 1300 2900 50  0001 C CNN
 	1    1300 2900
